Commit message: Updated robot model

File: ros_tank/urdf/gazebo.xacro (robot description, xacro)
@@ -2,5 +2,5 @@
 <robot>
     <!-- Colors -->
-    <gazebo reference="link_chassis">
+    <!-- <gazebo reference="link_chassis">
         <material>Gazebo/Blue</material>
     </gazebo>
@@ -24,19 +24,26 @@
         <mu1>0</mu1>
         <mu2>0</mu2>
+    </gazebo> -->
+    <gazebo reference="link_chassis">
+        <material>Gazebo/Blue</material>
     </gazebo>
-    <gazebo>
-        <plugin filename="libgazebo_ros_diff_drive.so" name="differential_drive_controller">
-            <alwaysOn>true</alwaysOn>
-            <updateRate>30</updateRate>
-            <leftJoint>joint_chassis_left_back_wheel</leftJoint>
-            <rightJoint>joint_chassis_right_back_wheel</rightJoint>
-            <wheelSeparation>0.6</wheelSeparation>
-            <wheelDiameter>0.3</wheelDiameter>
-            <torque>10</torque>
-            <commandTopic>cmd_vel</commandTopic>
-            <odometryTopic>odom</odometryTopic>
-            <odometryFrame>odom</odometryFrame>
-            <robotBaseFrame>link_chassis</robotBaseFrame>
-        </plugin>
+    <!-- Gazebo tags - Laser scan -->
+    <gazebo reference="joint_laser_scan_chassis">
+        <preserveFixedJoint>true</preserveFixedJoint>
+    </gazebo>
+    <gazebo reference="link_laser_scan">
+        <material>Gazebo/DarkGrey</material>
+    </gazebo>
+    <gazebo reference="joint_chassis_left_front_wheel">
+        <preserveFixedJoint>true</preserveFixedJoint>
+    </gazebo>
+    <gazebo reference="joint_chassis_left_rear_wheel">
+        <preserveFixedJoint>true</preserveFixedJoint>
+    </gazebo>
+    <gazebo reference="joint_chassis_right_front_wheel">
+        <preserveFixedJoint>true</preserveFixedJoint>
+    </gazebo>
+    <gazebo reference="joint_chassis_right_rear_wheel">
+        <preserveFixedJoint>true</preserveFixedJoint>
     </gazebo>
     <!-- Gazebo tags - Laser scan -->
@@ -79,5 +86,5 @@
     </gazebo>
     <gazebo reference="camera_link">
-        <sensor name="camera" type="camera">
+        <sensor name="camera_robot" type="camera">
             <camera>
                 <pose> 0 0 0 0 0 0 </pose>
@@ -100,3 +107,18 @@
         </sensor>
     </gazebo>
+    <!-- <gazebo>
+        <plugin filename="libgazebo_ros_diff_drive.so" name="differential_drive_controller">
+            <alwaysOn>true</alwaysOn>
+            <updateRate>20</updateRate>
+            <leftJoint>joint_chassis_left_middle_wheel</leftJoint>
+            <rightJoint>joint_chassis_right_middle_wheel</rightJoint>
+            <wheelSeparation>1.66</wheelSeparation>
+            <wheelDiameter>0.8</wheelDiameter>
+            <torque>10</torque>
+            <commandTopic>cmd_vel</commandTopic>
+            <odometryTopic>odom</odometryTopic>
+            <odometryFrame>odom</odometryFrame>
+            <robotBaseFrame>link_chassis</robotBaseFrame>
+        </plugin>
+    </gazebo> -->
 </robot>

File: ros_tank/urdf/robot.urdf (robot description, URDF)
Before this commit: robot robot, 7 links, 6 joints
Links:
- removed link link_front_left_wheel
- removed link link_front_right_wheel
- removed link link_middle_left_wheel
- removed link link_middle_right_wheel
- removed link link_rear_left_wheel
- removed link link_rear_right_wheel
- added link camera_link; visual box size=0.05 0.05 0.06
- added link link_laser_scan, mass 0.5; collision cylinder length=0.15 radius=0.1; visual cylinder length=0.15 radius=0.1
- added link link_left_back_wheel, mass 1; collision cylinder length=${length_cylinder_wheel} radius=${radius_cylinder_wheel}; collision cylinder length=${length_wheel} radius=${radius_wheel}
- added link link_left_front_wheel, mass 1; collision cylinder length=${length_cylinder_wheel} radius=${radius_cylinder_wheel}; collision cylinder length=${length_wheel} radius=${radius_wheel}
- added link link_right_back_wheel, mass 1; collision cylinder length=${length_cylinder_wheel} radius=${radius_cylinder_wheel}; collision cylinder length=${length_wheel} radius=${radius_wheel}
- added link link_right_front_wheel, mass 1; collision cylinder length=${length_cylinder_wheel} radius=${radius_cylinder_wheel}; collision cylinder length=${length_wheel} radius=${radius_wheel}
- link link_chassis: geometry collision box size=1 0.6 0.2; visual box size=1 0.6 0.2
Joints:
- removed joint joint_chassis_left_rear_wheel
- removed joint joint_chassis_left_wheel
- removed joint joint_chassis_right_rear_wheel
- removed joint joint_chassis_right_wheel
- added joint camera_joint: type fixed, parent link_chassis, child camera_link, origin xyz=0.45 0 0.13 rpy=0 0 0
- added joint joint_chassis_left_back_wheel: type continuous, parent link_chassis, child link_left_back_wheel, origin xyz=-0.45 0.28 0 rpy=0 0 0, axis 0 1 0, limit effort=10000 velocity=1000
- added joint joint_chassis_right_back_wheel: type continuous, parent link_chassis, child link_right_back_wheel, origin xyz=-0.45 -0.28 0 rpy=0 0 0, axis 0 1 0, limit effort=10000 velocity=1000
- added joint joint_laser_scan_chassis: type fixed, parent link_chassis, child link_laser_scan, origin xyz=0 0 0.16 rpy=0 0 0
- joint joint_chassis_left_front_wheel: child link_front_left_wheel -> link_left_front_wheel; origin xyz=0.065 0.077 -0.12 rpy=0 0 0 -> xyz=0.45 0.28 0 rpy=0 0 0; type fixed -> continuous
- joint joint_chassis_right_front_wheel: child link_front_right_wheel -> link_right_front_wheel; origin xyz=0.065 -0.077 -0.12 rpy=0 0 0 -> xyz=0.45 -0.28 0 rpy=0 0 0; type fixed -> continuous

File: ros_tank/urdf/robot.xacro (robot description, xacro)
@@ -1,5 +1,5 @@
 <?xml version="1.0" ?>
 <robot name="robot" xmlns:xacro="http://www.ros.org/wiki/xacro">
-    <xacro:include filename="$(find robot_project)/urdf/gazebo.xacro" />
+    <xacro:include filename="$(find ros_tank)/urdf/gazebo.xacro" />
     <!-- Parameters -->
     <xacro:property name="chassis_mass" value="10" />
@@ -8,215 +8,7 @@
     <xacro:property name="radius_cylinder_wheel" value="0.04" />
     <xacro:property name="length_cylinder_wheel" value="0.06" />
-    <!-- Gazebo tags - Laser scan -->
-    <gazebo reference="joint_laser_scan_chassis">
-        <preserveFixedJoint>true</preserveFixedJoint>
-    </gazebo>
-    <gazebo reference="link_laser_scan">
-        <material>Gazebo/DarkGrey</material>
-    </gazebo>
-    <!-- Link - chassis -->
-    <link name="link_chassis">
-        <inertial>
-            <mass value="10" />
-            <origin xyz="0 0 0.3" rpy="0 0 0" />
-            <inertia ixx="1.5417" ixy="0" ixz="0" iyy="3.467" iyz="0" izz="4.742" />
-        </inertial>
-        <collision>
-            <geometry>
-                <box size="1 0.6 0.2" />
-            </geometry>
-        </collision>
-        <visual>
-            <geometry>
-                <box size="1 0.6 0.2" />
-            </geometry>
-            <material name="DarkBlue">
-                <color rgba="0.2 0.2 0.4 1" />
-            </material>
-        </visual>
-    </link>
-    <joint name="joint_chassis_left_back_wheel" type="continuous">
-        <origin rpy="0 0 0" xyz="-0.45 0.28 0" />
-        <child link="link_left_back_wheel" />
-        <parent link="link_chassis" />
-        <axis rpy="0 0 0" xyz="0 1 0" />
-        <limit effort="10000" velocity="1000" />
-        <joint_properties damping="1.0" friction="1.0" />
-    </joint>
-    <link name="link_left_back_wheel">
-        <inertial>
-            <mass value="1" />
-            <origin xyz="0 0 0" rpy="0 0 0" />
-            <inertia ixx="0.002526666666667" ixy="0" ixz="0" iyy="0.002526666666667" iyz="0" izz="0.005"/>
-        </inertial>
-        <collision>
-            <origin rpy="1.5707 0 0" xyz="0 0.06 0" />
-            <geometry>
-                <cylinder length="${length_wheel}" radius="${radius_wheel}"/>
-            </geometry>
-        </collision>
-        <visual>
-            <origin rpy="1.5707 0 0" xyz="0 0.06 0" />
-            <geometry>
-                <cylinder length="${length_wheel}" radius="${radius_wheel}"/>
-            </geometry>
-            <material name="Black">
-                <color rgba="0.1 0.1 0.1 1" />
-            </material>
-        </visual>
-        <collision>
-            <origin rpy="1.5707 0 0" xyz="0 0.05 0" />
-            <geometry>
-                <cylinder length="${length_cylinder_wheel}" radius="${radius_cylinder_wheel}"/>
-            </geometry>
-        </collision>
-        <visual>
-            <origin rpy="1.5707 0 0" xyz="0 0.05 0" />
-            <geometry>
-                <cylinder length="${length_cylinder_wheel}" radius="${radius_cylinder_wheel}"/>
-            </geometry>
-            <material name="Black">
-                <color rgba="0.1 0.1 0.1 1" />
-            </material>
-        </visual>
-    </link>
-    <joint name="joint_chassis_right_back_wheel" type="continuous">
-        <origin rpy="0 0 0" xyz="-0.45 -0.28 0" />
-        <child link="link_right_back_wheel" />
-        <parent link="link_chassis" />
-        <axis rpy="0 0 0" xyz="0 1 0" />
-        <limit effort="10000" velocity="1000" />
-        <joint_properties damping="1.0" friction="1.0" />
-    </joint>
-    <link name="link_right_back_wheel">
-        <inertial>
-            <mass value="1" />
-            <origin xyz="0 0 0" rpy="0 0 0" />
-            <inertia ixx="0.002526666666667" ixy="0" ixz="0" iyy="0.002526666666667" iyz="0" izz="0.005"/>
-        </inertial>
-        <collision>
-            <origin rpy="1.5707 0 0" xyz="0 -0.06 0" />
-            <geometry>
-                <cylinder length="${length_wheel}" radius="${radius_wheel}"/>
-            </geometry>
-        </collision>
-        <visual>
-            <origin rpy="1.5707 0 0" xyz="0 -0.06 0" />
-            <geometry>
-                <cylinder length="${length_wheel}" radius="${radius_wheel}"/>
-            </geometry>
-            <material name="Black">
-                <color rgba="0.1 0.1 0.1 1" />
-            </material>
-        </visual>
-        <collision>
-            <origin rpy="1.5707 0 0" xyz="0 -0.05 0" />
-            <geometry>
-                <cylinder length="${length_cylinder_wheel}" radius="${radius_cylinder_wheel}"/>
-            </geometry>
-        </collision>
-        <visual>
-            <origin rpy="1.5707 0 0" xyz="0 -0.05 0" />
-            <geometry>
-                <cylinder length="${length_cylinder_wheel}" radius="${radius_cylinder_wheel}"/>
-            </geometry>
-            <material name="Black">
-                <color rgba="0.1 0.1 0.1 1" />
-            </material>
-        </visual>
-    </link>
-    <joint name="joint_chassis_left_front_wheel" type="continuous">
-        <origin rpy="0 0 0" xyz="0.45 0.28 0" />
-        <child link="link_left_front_wheel" />
-        <parent link="link_chassis" />
-        <axis rpy="0 0 0" xyz="0 1 0" />
-        <limit effort="10000" velocity="1000" />
-        <joint_properties damping="1.0" friction="1.0" />
-    </joint>
-    <link name="link_left_front_wheel">
-        <inertial>
-            <mass value="1" />
-            <origin xyz="0 0 0" rpy="0 0 0" />
-            <inertia ixx="0.002526666666667" ixy="0" ixz="0" iyy="0.002526666666667" iyz="0" izz="0.005"/>
-        </inertial>
-        <collision>
-            <origin rpy="1.5707 0 0" xyz="0 0.06 0" />
-            <geometry>
-                <cylinder length="${length_wheel}" radius="${radius_wheel}"/>
-            </geometry>
-        </collision>
-        <visual>
-            <origin rpy="1.5707 0 0" xyz="0 0.06 0" />
-            <geometry>
-                <cylinder length="${length_wheel}" radius="${radius_wheel}"/>
-            </geometry>
-            <material name="Black">
-                <color rgba="0.1 0.1 0.1 1" />
-            </material>
-        </visual>
-        <collision>
-            <origin rpy="1.5707 0 0" xyz="0 0.05 0" />
-            <geometry>
-                <cylinder length="${length_cylinder_wheel}" radius="${radius_cylinder_wheel}"/>
-            </geometry>
-        </collision>
-        <visual>
-            <origin rpy="1.5707 0 0" xyz="0 0.05 0" />
-            <geometry>
-                <cylinder length="${length_cylinder_wheel}" radius="${radius_cylinder_wheel}"/>
-            </geometry>
-            <material name="Black">
-                <color rgba="0.1 0.1 0.1 1" />
-            </material>
-        </visual>
-    </link>
-    <joint name="joint_chassis_right_front_wheel" type="continuous">
-        <origin rpy="0 0 0" xyz="0.45 -0.28 0" />
-        <child link="link_right_front_wheel" />
-        <parent link="link_chassis" />
-        <axis rpy="0 0 0" xyz="0 1 0" />
-        <limit effort="10000" velocity="1000" />
-        <joint_properties damping="1.0" friction="1.0" />
-    </joint>
-    <link name="link_right_front_wheel">
-        <inertial>
-            <mass value="1" />
-            <origin xyz="0 0 0" rpy="0 0 0" />
-            <inertia ixx="0.002526666666667" ixy="0" ixz="0" iyy="0.002526666666667" iyz="0" izz="0.005"/>
-        </inertial>
-        <collision>
-            <origin rpy="1.5707 0 0" xyz="0 -0.06 0" />
-            <geometry>
-                <cylinder length="${length_wheel}" radius="${radius_wheel}"/>
-            </geometry>
-        </collision>
-        <visual>
-            <origin rpy="1.5707 0 0" xyz="0 -0.06 0" />
-            <geometry>
-                <cylinder length="${length_wheel}" radius="${radius_wheel}"/>
-            </geometry>
-            <material name="Black">
-                <color rgba="0.1 0.1 0.1 1" />
-            </material>
-        </visual>
-        <collision>
-            <origin rpy="1.5707 0 0" xyz="0 -0.05 0" />
-            <geometry>
-                <cylinder length="${length_cylinder_wheel}" radius="${radius_cylinder_wheel}"/>
-            </geometry>
-        </collision>
-        <visual>
-            <origin rpy="1.5707 0 0" xyz="0 -0.05 0" />
-            <geometry>
-                <cylinder length="${length_cylinder_wheel}" radius="${radius_cylinder_wheel}"/>
-            </geometry>
-            <material name="Black">
-                <color rgba="0.1 0.1 0.1 1" />
-            </material>
-        </visual>
-    </link>
     <!-- Laser scan -->
     <joint name="joint_laser_scan_chassis" type="fixed">
-        <origin rpy="0 0 0" xyz="0 0 0.16" />
+        <origin rpy="0 0 0" xyz="-0.01 0 0.11" />
         <child link="link_laser_scan" />
         <parent link="link_chassis" />
@@ -232,5 +24,6 @@
             <origin xyz="0 0 0" rpy="0 0 0" />
             <geometry>
-                <cylinder radius="0.1" length="0.15"/>
+                <mesh filename="package://ros_tank/meshes/lidarA1.stl" pose="0 0 0" scale="0.00111 0.00111 0.0011"/>
+                <!-- <cylinder radius="0.04" length="0.04"/> -->
             </geometry>
             <material name="Red">
@@ -241,5 +34,5 @@
             <origin xyz="0 0 0" rpy="0 0 0"/>
             <geometry>
-                <cylinder radius="0.1" length="0.15"/>
+                <cylinder radius="0.2" length="0.1"/>
             </geometry>
         </collision>
@@ -249,10 +42,202 @@
         <parent link="link_chassis"/>
         <child link="camera_link"/>
-        <origin xyz="0.45 0 0.13" rpy="0 0 0"/>
+        <origin xyz="0.11 0 0.04" rpy="0 0 0"/>
     </joint>
     <link name="camera_link">
         <visual>
             <geometry>
-                <box size="0.05 0.05 0.06"/>
+                <mesh filename="package://ros_tank/meshes/camera.stl" pose="0 0 0" scale="0.00111 0.00111 0.0011"/>
+                <!-- <box size="0.02 0.08 0.038"/> -->
+            </geometry>
+        </visual>
+    </link>
+    <!-- Link - chassis -->
+    <link name="link_chassis">
+        <inertial>
+            <mass value="10" />
+            <origin xyz="0 0 0.3" rpy="0 0 0" />
+            <inertia ixx="1.5417" ixy="0" ixz="0" iyy="3.467" iyz="0" izz="4.742" />
+        </inertial>
+        <visual>
+            <geometry>
+                <!-- <box size="0.22 0.14 0.25" /> -->
+                <mesh filename="package://ros_tank/meshes/tank_body.stl" pose="0 0 0" scale="0.00111 0.00111 0.0011"/>
+            </geometry>
+            <material name="Red">
+                <color rgba="1 0 0 1" />
+            </material>
+        </visual>
+    </link>
+    <!-- Joint - chassis / left front wheel -->
+    <joint name="joint_chassis_left_front_wheel" type="fixed">
+        <origin rpy="0 0 0" xyz="0.065 0.077 -0.12" />
+        <child link="link_front_left_wheel" />
+        <parent link="link_chassis" />
+        <axis rpy="0 0 0" xyz="0 1 0" />
+        <limit effort="10000" velocity="1000" />
+        <joint_properties damping="1.0" friction="1.0" />
+    </joint>
+    <!-- Link - left front wheel -->
+    <link name="link_front_left_wheel">
+        <inertial>
+            <mass value="10" />
+            <origin xyz="0 0 0.3" rpy="0 0 0" />
+            <inertia ixx="1.5417" ixy="0" ixz="0" iyy="3.467" iyz="0" izz="4.742" />
+        </inertial>
+        <collision>
+            <origin rpy="1.5707 0 0" xyz="0 -0.015 0" />
+            <geometry>
+                <cylinder length="0.03" radius="0.02"/>
+            </geometry>
+        </collision>
+        <visual>
+            <origin rpy="1.5707 0 0" xyz="0 0.015 0" />
+            <geometry>
+                <cylinder length="0.03" radius="0.02"/>
+            </geometry>
+        </visual>
+    </link>
+    <!-- Joint - chassis / left middle wheel -->
+    <joint name="joint_chassis_left_middle_wheel" type="continuous">
+        <origin rpy="0 0 0" xyz="0 0.077 -0.12" />
+        <child link="link_middle_left_wheel" />
+        <parent link="link_chassis" />
+        <axis rpy="0 0 0" xyz="0 1 0" />
+        <limit effort="10000" velocity="1000" />
+        <joint_properties damping="1.0" friction="1.0" />
+    </joint>
+    <!-- Link - left middle wheel -->
+    <link name="link_middle_left_wheel">
+        <inertial>
+            <mass value="10" />
+            <origin xyz="0 0 0.3" rpy="0 0 0" />
+            <inertia ixx="1.5417" ixy="0" ixz="0" iyy="3.467" iyz="0" izz="4.742" />
+        </inertial>
+        <collision>
+            <origin rpy="1.5707 0 0" xyz="0 0.015 0" />
+            <geometry>
+                <cylinder length="0.03" radius="0.02"/>
+            </geometry>
+        </collision>
+        <visual>
+            <origin rpy="1.5707 0 0" xyz="0 0.015 0" />
+            <geometry>
+                <cylinder length="0.03" radius="0.02"/>
+            </geometry>
+        </visual>
+    </link>
+    <!-- Joint - chassis / left rear wheel -->
+    <joint name="joint_chassis_left_rear_wheel" type="fixed">
+        <origin rpy="0 0 0" xyz="-0.065 0.077 -0.12" />
+        <child link="link_rear_left_wheel" />
+        <parent link="link_chassis" />
+        <axis rpy="0 0 0" xyz="0 1 0" />
+        <limit effort="10000" velocity="1000" />
+        <joint_properties damping="1.0" friction="1.0" />
+    </joint>
+    <!-- Link - left rear wheel -->
+    <link name="link_rear_left_wheel">
+        <inertial>
+            <mass value="10" />
+            <origin xyz="0 0 0.3" rpy="0 0 0" />
+            <inertia ixx="1.5417" ixy="0" ixz="0" iyy="3.467" iyz="0" izz="4.742" />
+        </inertial>
+        <collision>
+            <origin rpy="1.5707 0 0" xyz="0 0.015 0" />
+            <geometry>
+                <cylinder length="0.03" radius="0.02"/>
+            </geometry>
+        </collision>
+        <visual>
+            <origin rpy="1.5707 0 0" xyz="0 0.015 0" />
+            <geometry>
+                <cylinder length="0.03" radius="0.02"/>
+            </geometry>
+        </visual>
+    </link>
+    <!-- Joint - chassis / right front wheel -->
+    <joint name="joint_chassis_right_front_wheel" type="fixed">
+        <origin rpy="0 0 0" xyz="0.065 -0.077 -0.12" />
+        <child link="link_front_right_wheel" />
+        <parent link="link_chassis" />
+        <axis rpy="0 0 0" xyz="0 1 0" />
+        <limit effort="10000" velocity="1000" />
+        <joint_properties damping="1.0" friction="1.0" />
+    </joint>
+    <!-- Link - right front wheel -->
+    <link name="link_front_right_wheel">
+        <inertial>
+            <mass value="10" />
+            <origin xyz="0 0 0.3" rpy="0 0 0" />
+            <inertia ixx="1.5417" ixy="0" ixz="0" iyy="3.467" iyz="0" izz="4.742" />
+        </inertial>
+        <collision>
+            <origin rpy="1.5707 0 0" xyz="0 -0.015 0" />
+            <geometry>
+                <cylinder length="0.03" radius="0.02"/>
+            </geometry>
+        </collision>
+        <visual>
+            <origin rpy="1.5707 0 0" xyz="0 -0.015 0" />
+            <geometry>
+                <cylinder length="0.03" radius="0.02"/>
+            </geometry>
+        </visual>
+    </link>
+    <!-- Joint - chassis / right middle wheel -->
+    <joint name="joint_chassis_right_middle_wheel" type="continuous">
+        <origin rpy="0 0 0" xyz="0 -0.077 -0.12" />
+        <child link="link_middle_right_wheel" />
+        <parent link="link_chassis" />
+        <axis rpy="0 0 0" xyz="0 1 0" />
+        <limit effort="10000" velocity="1000" />
+        <joint_properties damping="1.0" friction="1.0" />
+    </joint>
+    <!-- Link - right middle wheel -->
+    <link name="link_middle_right_wheel">
+        <inertial>
+            <mass value="10" />
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