Commit message: Update config

File: ros_tank/urdf/gazebo.xacro (robot description, xacro)
@@ -2,27 +2,27 @@
 <robot>
     <!-- Colors -->
-    <!-- <gazebo reference="link_chassis">
+    <gazebo reference="link_chassis">
         <material>Gazebo/Blue</material>
     </gazebo>
-    <gazebo reference="link_left_back_wheel">
+    <gazebo reference="link_front_left_wheel">
         <material>Gazebo/Black</material>
         <mu1>0.1</mu1>
         <mu2>0.1</mu2>
     </gazebo>
-    <gazebo reference="link_right_back_wheel">
+    <gazebo reference="link_rear_right_wheel">
         <material>Gazebo/Black</material>
         <mu1>0.1</mu1>
         <mu2>0.1</mu2>
     </gazebo>
-    <gazebo reference="link_left_front_wheel">
+    <gazebo reference="link_rear_left_wheel">
         <material>Gazebo/Black</material>
         <mu1>0</mu1>
         <mu2>0</mu2>
     </gazebo>
-    <gazebo reference="link_right_front_wheel">
+    <gazebo reference="link_front_right_wheel">
         <material>Gazebo/Black</material>
         <mu1>0</mu1>
         <mu2>0</mu2>
-    </gazebo> -->
+    </gazebo>
     <gazebo reference="link_chassis">
         <material>Gazebo/Blue</material>
@@ -107,5 +107,5 @@
         </sensor>
     </gazebo>
-    <!-- <gazebo>
+    <gazebo>
         <plugin filename="libgazebo_ros_diff_drive.so" name="differential_drive_controller">
             <alwaysOn>true</alwaysOn>
@@ -121,4 +121,4 @@
             <robotBaseFrame>link_chassis</robotBaseFrame>
         </plugin>
-    </gazebo> -->
+    </gazebo>
 </robot>

File: ros_tank/urdf/robot.xacro (robot description, xacro)
@@ -2,10 +2,4 @@
 <robot name="robot" xmlns:xacro="http://www.ros.org/wiki/xacro">
     <xacro:include filename="$(find ros_tank)/urdf/gazebo.xacro" />
-    <!-- Parameters -->
-    <xacro:property name="chassis_mass" value="10" />
-    <xacro:property name="radius_wheel" value="0.15" />
-    <xacro:property name="length_wheel" value="0.06" />
-    <xacro:property name="radius_cylinder_wheel" value="0.04" />
-    <xacro:property name="length_cylinder_wheel" value="0.06" />
     <!-- Laser scan -->
     <joint name="joint_laser_scan_chassis" type="fixed">

Commit message: Updated config

File: ros_tank/urdf/gazebo.xacro (robot description, xacro)
@@ -107,5 +107,5 @@
         </sensor>
     </gazebo>
-    <gazebo>
+    <!-- <gazebo>
         <plugin filename="libgazebo_ros_diff_drive.so" name="differential_drive_controller">
             <alwaysOn>true</alwaysOn>
@@ -116,9 +116,17 @@
             <wheelDiameter>0.8</wheelDiameter>
             <torque>10</torque>
+            <wheelTorque>5</wheelTorque>
             <commandTopic>cmd_vel</commandTopic>
             <odometryTopic>odom</odometryTopic>
             <odometryFrame>odom</odometryFrame>
             <robotBaseFrame>link_chassis</robotBaseFrame>
+            <publishWheelTF>true</publishWheelTF>
+            <publishWheelJointState>true</publishWheelJointState>
+            <publishOdomTF>true</publishOdomTF>
+            <wheelAcceleration>0</wheelAcceleration>
+            <odometrySource>world</odometrySource>
+            <publishTf>1</publishTf>
+            <rosDebugLevel>na</rosDebugLevel>
         </plugin>
-    </gazebo>
+    </gazebo> -->
 </robot>

File: ros_tank/urdf/robot.xacro (robot description, xacro)
@@ -28,5 +28,5 @@
             <origin xyz="0 0 0" rpy="0 0 0"/>
             <geometry>
-                <cylinder radius="0.2" length="0.1"/>
+                <cylinder radius="0.04" length="0.04"/>
             </geometry>
         </collision>
@@ -48,9 +48,4 @@
     <!-- Link - chassis -->
     <link name="link_chassis">
-        <inertial>
-            <mass value="10" />
-            <origin xyz="0 0 0.3" rpy="0 0 0" />
-            <inertia ixx="1.5417" ixy="0" ixz="0" iyy="3.467" iyz="0" izz="4.742" />
-        </inertial>
         <visual>
             <geometry>

Commit message: Fix for urdf

File: ros_tank/urdf/gazebo.xacro (robot description, xacro)
@@ -7,11 +7,11 @@
     <gazebo reference="link_front_left_wheel">
         <material>Gazebo/Black</material>
-        <mu1>0.1</mu1>
-        <mu2>0.1</mu2>
+        <mu1>0</mu1>
+        <mu2>0</mu2>
     </gazebo>
     <gazebo reference="link_rear_right_wheel">
         <material>Gazebo/Black</material>
-        <mu1>0.1</mu1>
-        <mu2>0.1</mu2>
+        <mu1>0</mu1>
+        <mu2>0</mu2>
     </gazebo>
     <gazebo reference="link_rear_left_wheel">
@@ -25,15 +25,22 @@
         <mu2>0</mu2>
     </gazebo>
-    <gazebo reference="link_chassis">
-        <material>Gazebo/Blue</material>
+    <gazebo reference="link_middle_right_wheel">
+        <material>Gazebo/Black</material>
+        <mu1>0.1</mu1>
+        <mu2>0.1</mu2>
+    </gazebo>
+    <gazebo reference="link_middle_left_wheel">
+        <material>Gazebo/Black</material>
+        <mu1>0.1</mu1>
+        <mu2>0.1</mu2>
     </gazebo>
     <!-- Gazebo tags - Laser scan -->
-    <gazebo reference="joint_laser_scan_chassis">
+    <!-- <gazebo reference="joint_laser_scan_chassis">
         <preserveFixedJoint>true</preserveFixedJoint>
-    </gazebo>
+    </gazebo> -->
     <gazebo reference="link_laser_scan">
         <material>Gazebo/DarkGrey</material>
     </gazebo>
-    <gazebo reference="joint_chassis_left_front_wheel">
+    <!-- <gazebo reference="joint_chassis_left_front_wheel">
         <preserveFixedJoint>true</preserveFixedJoint>
     </gazebo>
@@ -47,11 +54,5 @@
         <preserveFixedJoint>true</preserveFixedJoint>
     </gazebo>
-    <!-- Gazebo tags - Laser scan -->
-    <gazebo reference="joint_laser_scan_chassis">
-        <preserveFixedJoint>true</preserveFixedJoint>
-    </gazebo>
-    <gazebo reference="link_laser_scan">
-        <material>Gazebo/DarkGrey</material>
-    </gazebo>
+     -->
     <gazebo reference="link_laser_scan">
         <sensor type="ray" name="head_hokuyo_sensor">
@@ -107,5 +108,5 @@
         </sensor>
     </gazebo>
-    <!-- <gazebo>
+    <gazebo>
         <plugin filename="libgazebo_ros_diff_drive.so" name="differential_drive_controller">
             <alwaysOn>true</alwaysOn>
@@ -113,6 +114,6 @@
             <leftJoint>joint_chassis_left_middle_wheel</leftJoint>
             <rightJoint>joint_chassis_right_middle_wheel</rightJoint>
-            <wheelSeparation>1.66</wheelSeparation>
-            <wheelDiameter>0.8</wheelDiameter>
+            <wheelSeparation>0.14</wheelSeparation>
+            <wheelDiameter>0.04</wheelDiameter>
             <torque>10</torque>
             <wheelTorque>5</wheelTorque>
@@ -121,12 +122,12 @@
             <odometryFrame>odom</odometryFrame>
             <robotBaseFrame>link_chassis</robotBaseFrame>
-            <publishWheelTF>true</publishWheelTF>
-            <publishWheelJointState>true</publishWheelJointState>
+            <publishWheelTF>false</publishWheelTF>
+            <publishWheelJointState>false</publishWheelJointState>
             <publishOdomTF>true</publishOdomTF>
             <wheelAcceleration>0</wheelAcceleration>
+            <rosDebugLevel>na</rosDebugLevel>
             <odometrySource>world</odometrySource>
             <publishTf>1</publishTf>
-            <rosDebugLevel>na</rosDebugLevel>
         </plugin>
-    </gazebo> -->
+    </gazebo>
 </robot>

File: ros_tank/urdf/robot.xacro (robot description, xacro)
@@ -39,4 +39,10 @@
     </joint>
     <link name="camera_link">
+        <collision>
+            <origin xyz="0 0 0" rpy="0 0 0"/>
+            <geometry>
+                <box size="0.02 0.08 0.038"/>
+            </geometry>
+        </collision>
         <visual>
             <geometry>
@@ -48,4 +54,10 @@
     <!-- Link - chassis -->
     <link name="link_chassis">
+        <collision>
+            <origin xyz="0 0 0" rpy="0 0 0"/>
+            <geometry>
+                <box size="0.22 0.14 0.25" />
+            </geometry>
+        </collision>
         <visual>
             <geometry>
