Commit message: Added meshes to camera

File: ros_tank/urdf/robot.xacro (robot description, xacro)
@@ -34,7 +34,7 @@
     <!-- Camera -->
     <joint name="camera_joint" type="fixed">
-        <parent link="link_chassis"/>
+        <parent link="camera_second_servo_link"/>
         <child link="camera_link"/>
-        <origin xyz="0.11 0 0.04" rpy="0 0 0"/>
+        <origin xyz="0.024 0 0.017" rpy="0 0 0"/>
     </joint>
     <link name="camera_link">
@@ -244,3 +244,53 @@
         </visual>
     </link>
+     <!-- Joint - camera second servo -->
+    <joint name="camera_servo_second_joint" type="revolute">
+        <origin xyz="0.03 -0.005 0.02" rpy="0 0 0"/>
+        <parent link="camera_servo_first_link"/>
+        <child link="camera_second_servo_link"/>
+        <axis xyz="0 1 0"/>
+        <limit lower="-1.15" upper="1.4" velocity="100" effort="100"/>
+    </joint>
+    <!-- Link - camera second servo -->
+    <link name="camera_second_servo_link">
+        <visual>
+            <origin xyz="0 0 0" rpy="0 0 0"/>
+            <geometry>
+                <!-- <box size="0.02 0.03 0.03" /> -->
+                <mesh filename="package://ros_tank/meshes/camera_servo_2.stl" pose="0 0 0" scale="0.0011 0.00111 0.0011"/>
+            </geometry>
+            <material name="orange" />
+        </visual>
+        <collision>
+            <origin xyz="0 0 0" rpy="0 0 0"/>
+            <geometry>
+                <box size="0.02 0.03 0.03" />
+            </geometry>
+        </collision>
+    </link>
+     <!-- Joint - camera first servo -->
+    <joint name="camera_servo_first_joint" type="revolute">
+        <origin xyz="0.053 0 0" rpy="0 0 0"/>
+        <parent link="link_chassis"/>
+        <child link="camera_servo_first_link"/>
+        <axis xyz="0 0 1"/>
+        <limit lower="-1.15" upper="1.4" velocity="100" effort="100"/>
+    </joint>
+    <!-- Link - camera first servo -->
+    <link name="camera_servo_first_link">
+        <visual>
+            <origin xyz="0 0 0" rpy="0 0 0"/>
+            <geometry>
+                <mesh filename="package://ros_tank/meshes/camera_servo_1.stl" pose="0 0 0" scale="0.0011 0.00111 0.0011"/>
+                <!-- <box size="0.03 0.04 0.05" /> -->
+            </geometry>
+            <material name="orange" />
+        </visual>
+        <collision>
+            <origin xyz="0 0 0" rpy="0 0 0"/>
+            <geometry>
+                <box size="0.03 0.04 0.05" />
+            </geometry>
+        </collision>
+    </link>
 </robot>

Commit message: Added moveit

File: ros_tank/urdf/robot.xacro (robot description, xacro)
@@ -2,4 +2,10 @@
 <robot name="robot" xmlns:xacro="http://www.ros.org/wiki/xacro">
     <xacro:include filename="$(find ros_tank)/urdf/gazebo.xacro" />
+    <link name="world"></link>
+    <joint name="joint_world" type="fixed">
+        <origin rpy="0 0 0" xyz="0 0 0" />
+        <child link="link_chassis" />
+        <parent link="world" />
+    </joint>
     <!-- Laser scan -->
     <joint name="joint_laser_scan_chassis" type="fixed">
@@ -28,5 +34,6 @@
             <origin xyz="0 0 0" rpy="0 0 0"/>
             <geometry>
-                <cylinder radius="0.04" length="0.04"/>
+                <mesh filename="package://ros_tank/meshes/lidarA1.stl" pose="0 0 0" scale="0.00111 0.00111 0.0011"/>
+                <!-- <cylinder radius="0.04" length="0.04"/> -->
             </geometry>
         </collision>
@@ -36,18 +43,19 @@
         <parent link="camera_second_servo_link"/>
         <child link="camera_link"/>
-        <origin xyz="0.024 0 0.017" rpy="0 0 0"/>
+        <origin xyz="0.03 0 0.017" rpy="0 0 0"/>
     </joint>
     <link name="camera_link">
         <collision>
             <origin xyz="0 0 0" rpy="0 0 0"/>
-            <geometry>
-                <box size="0.02 0.08 0.038"/>
-            </geometry>
-        </collision>
-        <visual>
             <geometry>
                 <mesh filename="package://ros_tank/meshes/camera.stl" pose="0 0 0" scale="0.00111 0.00111 0.0011"/>
                 <!-- <box size="0.02 0.08 0.038"/> -->
             </geometry>
+        </collision>
+        <visual>
+            <geometry>
+                <mesh filename="package://ros_tank/meshes/camera.stl" pose="0 0 0" scale="0.00111 0.00111 0.0011"/>
+                <!-- <box size="0.02 0.08 0.038"/> -->
+            </geometry>
         </visual>
     </link>
@@ -57,5 +65,6 @@
             <origin xyz="0 0 0" rpy="0 0 0"/>
             <geometry>
-                <box size="0.22 0.14 0.25" />
+                <!-- <box size="0.22 0.14 0.25" /> -->
+                <mesh filename="package://ros_tank/meshes/tank_body.stl" pose="0 0 0" scale="0.00111 0.00111 0.0011"/>
             </geometry>
         </collision>
@@ -265,5 +274,6 @@
             <origin xyz="0 0 0" rpy="0 0 0"/>
             <geometry>
-                <box size="0.02 0.03 0.03" />
+                <!-- <box size="0.02 0.03 0.03" /> -->
+                <mesh filename="package://ros_tank/meshes/camera_servo_2.stl" pose="0 0 0" scale="0.0011 0.00111 0.0011"/>
             </geometry>
         </collision>
@@ -290,5 +300,6 @@
             <origin xyz="0 0 0" rpy="0 0 0"/>
             <geometry>
-                <box size="0.03 0.04 0.05" />
+                <mesh filename="package://ros_tank/meshes/camera_servo_1.stl" pose="0 0 0" scale="0.0011 0.00111 0.0011"/>
+                <!-- <box size="0.03 0.04 0.05" /> -->
             </geometry>
         </collision>

Commit message: Fix for collisions

File: ros_tank/urdf/robot.xacro (robot description, xacro)
@@ -34,6 +34,5 @@
             <origin xyz="0 0 0" rpy="0 0 0"/>
             <geometry>
-                <mesh filename="package://ros_tank/meshes/lidarA1.stl" pose="0 0 0" scale="0.00111 0.00111 0.0011"/>
-                <!-- <cylinder radius="0.04" length="0.04"/> -->
+                <cylinder radius="0.04" length="0.04"/>
             </geometry>
         </collision>
@@ -49,13 +48,12 @@
             <origin xyz="0 0 0" rpy="0 0 0"/>
             <geometry>
+                <box size="0.02 0.08 0.038"/>
+            </geometry>
+        </collision>
+        <visual>
+            <geometry>
                 <mesh filename="package://ros_tank/meshes/camera.stl" pose="0 0 0" scale="0.00111 0.00111 0.0011"/>
                 <!-- <box size="0.02 0.08 0.038"/> -->
             </geometry>
-        </collision>
-        <visual>
-            <geometry>
-                <mesh filename="package://ros_tank/meshes/camera.stl" pose="0 0 0" scale="0.00111 0.00111 0.0011"/>
-                <!-- <box size="0.02 0.08 0.038"/> -->
-            </geometry>
         </visual>
     </link>
@@ -63,8 +61,7 @@
     <link name="link_chassis">
         <collision>
-            <origin xyz="0 0 0" rpy="0 0 0"/>
-            <geometry>
-                <!-- <box size="0.22 0.14 0.25" /> -->
-                <mesh filename="package://ros_tank/meshes/tank_body.stl" pose="0 0 0" scale="0.00111 0.00111 0.0011"/>
+            <origin xyz="0 0 -0.08" rpy="0 0 0"/>
+            <geometry>
+                <box size="0.25 0.25 0.1" />
             </geometry>
         </collision>
@@ -263,4 +260,10 @@
     <!-- Link - camera second servo -->
     <link name="camera_second_servo_link">
+        <collision>
+            <origin xyz="0 0 0.01" rpy="0 0 0"/>
+            <geometry>
+                <box size="0.02 0.03 0.03" />
+            </geometry>
+        </collision>
         <visual>
             <origin xyz="0 0 0" rpy="0 0 0"/>
@@ -271,11 +274,4 @@
             <material name="orange" />
         </visual>
-        <collision>
-            <origin xyz="0 0 0" rpy="0 0 0"/>
-            <geometry>
-                <!-- <box size="0.02 0.03 0.03" /> -->
-                <mesh filename="package://ros_tank/meshes/camera_servo_2.stl" pose="0 0 0" scale="0.0011 0.00111 0.0011"/>
-            </geometry>
-        </collision>
     </link>
      <!-- Joint - camera first servo -->
@@ -289,4 +285,10 @@
     <!-- Link - camera first servo -->
     <link name="camera_servo_first_link">
+        <collision>
+            <origin xyz="0 0 -0.005" rpy="0 0 0"/>
+            <geometry>
+                <box size="0.03 0.04 0.03" />
+            </geometry>
+        </collision>
         <visual>
             <origin xyz="0 0 0" rpy="0 0 0"/>
@@ -297,11 +299,4 @@
             <material name="orange" />
         </visual>
-        <collision>
-            <origin xyz="0 0 0" rpy="0 0 0"/>
-            <geometry>
-                <mesh filename="package://ros_tank/meshes/camera_servo_1.stl" pose="0 0 0" scale="0.0011 0.00111 0.0011"/>
-                <!-- <box size="0.03 0.04 0.05" /> -->
-            </geometry>
-        </collision>
     </link>
 </robot>

Commit message: Update Dockerfile and spawn launch

File: ros_tank/urdf/robot.xacro (robot description, xacro)
@@ -1,6 +1,24 @@
 <?xml version="1.0" ?>
 <robot name="robot" xmlns:xacro="http://www.ros.org/wiki/xacro">
-    <xacro:include filename="$(find ros_tank)/urdf/gazebo.xacro" />
+    <!-- <xacro:include filename="$(find ros_tank)/urdf/gazebo.xacro" /> -->
     <link name="world"></link>
+    <!-- Link - chassis -->
+    <link name="link_chassis">
+        <collision>
+            <origin xyz="0 0 -0.08" rpy="0 0 0"/>
+            <geometry>
+                <box size="0.25 0.25 0.1" />
+            </geometry>
+        </collision>
+        <visual>
+            <geometry>
+                <!-- <box size="0.22 0.14 0.25" /> -->
+                <mesh filename="package://ros_tank/meshes/tank_body.stl" pose="0 0 0" scale="0.00111 0.00111 0.0011"/>
+            </geometry>
+            <material name="Red">
+                <color rgba="1 0 0 1" />
+            </material>
+        </visual>
+    </link>
     <joint name="joint_world" type="fixed">
         <origin rpy="0 0 0" xyz="0 0 0" />
@@ -39,4 +57,18 @@
     </link>
     <!-- Camera -->
+    <link name="camera_link">
+        <collision>
+            <origin xyz="0 0 0" rpy="0 0 0"/>
+            <geometry>
+                <box size="0.02 0.08 0.038"/>
+            </geometry>
+        </collision>
+        <visual>
+            <geometry>
+                <mesh filename="package://ros_tank/meshes/camera.stl" pose="0 0 0" scale="0.00111 0.00111 0.0011"/>
+                <!-- <box size="0.02 0.08 0.038"/> -->
+            </geometry>
+        </visual>
+    </link>
     <joint name="camera_joint" type="fixed">
         <parent link="camera_second_servo_link"/>
@@ -44,34 +76,22 @@
         <origin xyz="0.03 0 0.017" rpy="0 0 0"/>
     </joint>
-    <link name="camera_link">
-        <collision>
-            <origin xyz="0 0 0" rpy="0 0 0"/>
-            <geometry>
-                <box size="0.02 0.08 0.038"/>
-            </geometry>
-        </collision>
-        <visual>
-            <geometry>
-                <mesh filename="package://ros_tank/meshes/camera.stl" pose="0 0 0" scale="0.00111 0.00111 0.0011"/>
-                <!-- <box size="0.02 0.08 0.038"/> -->
-            </geometry>
-        </visual>
-    </link>
-    <!-- Link - chassis -->
-    <link name="link_chassis">
-        <collision>
-            <origin xyz="0 0 -0.08" rpy="0 0 0"/>
-            <geometry>
-                <box size="0.25 0.25 0.1" />
-            </geometry>
-        </collision>
-        <visual>
-            <geometry>
-                <!-- <box size="0.22 0.14 0.25" /> -->
-                <mesh filename="package://ros_tank/meshes/tank_body.stl" pose="0 0 0" scale="0.00111 0.00111 0.0011"/>
-            </geometry>
-            <material name="Red">
-                <color rgba="1 0 0 1" />
-            </material>
+    <!-- Link - left front wheel -->
+    <link name="link_front_left_wheel">
+        <inertial>
+            <mass value="10" />
+            <origin xyz="0 0 0.3" rpy="0 0 0" />
+            <inertia ixx="1.5417" ixy="0" ixz="0" iyy="3.467" iyz="0" izz="4.742" />
+        </inertial>
+        <collision>
+            <origin rpy="1.5707 0 0" xyz="0 -0.015 0" />
+            <geometry>
+                <cylinder length="0.03" radius="0.02"/>
+            </geometry>
+        </collision>
+        <visual>
+            <origin rpy="1.5707 0 0" xyz="0 0.015 0" />
+            <geometry>
+                <cylinder length="0.03" radius="0.02"/>
+            </geometry>
         </visual>
     </link>
@@ -85,13 +105,13 @@
         <joint_properties damping="1.0" friction="1.0" />
     </joint>
-    <!-- Link - left front wheel -->
-    <link name="link_front_left_wheel">
-        <inertial>
-            <mass value="10" />
-            <origin xyz="0 0 0.3" rpy="0 0 0" />
-            <inertia ixx="1.5417" ixy="0" ixz="0" iyy="3.467" iyz="0" izz="4.742" />
-        </inertial>
-        <collision>
-            <origin rpy="1.5707 0 0" xyz="0 -0.015 0" />
+    <!-- Link - left middle wheel -->
+    <link name="link_middle_left_wheel">
+        <inertial>
+            <mass value="10" />
+            <origin xyz="0 0 0.3" rpy="0 0 0" />
+            <inertia ixx="1.5417" ixy="0" ixz="0" iyy="3.467" iyz="0" izz="4.742" />
+        </inertial>
+        <collision>
+            <origin rpy="1.5707 0 0" xyz="0 0.015 0" />
             <geometry>
                 <cylinder length="0.03" radius="0.02"/>
@@ -114,6 +134,6 @@
         <joint_properties damping="1.0" friction="1.0" />
     </joint>
-    <!-- Link - left middle wheel -->
-    <link name="link_middle_left_wheel">
+    <!-- Link - left rear wheel -->
+    <link name="link_rear_left_wheel">
         <inertial>
             <mass value="10" />
@@ -143,24 +163,4 @@
         <joint_properties damping="1.0" friction="1.0" />
     </joint>
-    <!-- Link - left rear wheel -->
-    <link name="link_rear_left_wheel">
-        <inertial>
-            <mass value="10" />
-            <origin xyz="0 0 0.3" rpy="0 0 0" />
-            <inertia ixx="1.5417" ixy="0" ixz="0" iyy="3.467" iyz="0" izz="4.742" />
-        </inertial>
-        <collision>
-            <origin rpy="1.5707 0 0" xyz="0 0.015 0" />
-            <geometry>
-                <cylinder length="0.03" radius="0.02"/>
-            </geometry>
-        </collision>
-        <visual>
-            <origin rpy="1.5707 0 0" xyz="0 0.015 0" />
-            <geometry>
-                <cylinder length="0.03" radius="0.02"/>
-            </geometry>
-        </visual>
-    </link>
     <!-- Joint - chassis / right front wheel -->
     <joint name="joint_chassis_right_front_wheel" type="fixed">
