Commit message: Added gazebo.xacro

File: ros_tank_description/urdf/gazebo.xacro (robot description, xacro)
@@ -1,18 +1,158 @@
-    <!-- <gazebo reference="joint_chassis_left_front_wheel">
+<?xml version="1.0"?>
+<robot>
+    <gazebo reference="link_laser_scan">
+        <material>Gazebo/Red</material>
+    </gazebo>
+    <gazebo reference="link_chassis">
+        <material>Gazebo/DarkGrey</material>
+    </gazebo>
+    <gazebo reference="camera_servo_first_link">
+        <material>Gazebo/Red</material>
+    </gazebo>
+    <gazebo reference="camera_link">
+        <material>Gazebo/Red</material>
+    </gazebo>
+    <gazebo reference="camera_second_servo_link">
+        <material>Gazebo/Blue</material>
+    </gazebo>
+    <gazebo reference="joint_laser_scan_chassis">
         <preserveFixedJoint>true</preserveFixedJoint>
     </gazebo>
-    <gazebo reference="joint_chassis_left_rear_wheel">
+    <gazebo reference="camera_servo_first_joint">
         <preserveFixedJoint>true</preserveFixedJoint>
     </gazebo>
-    <gazebo reference="joint_chassis_right_front_wheel">
+    <gazebo reference="camera_servo_second_joint">
         <preserveFixedJoint>true</preserveFixedJoint>
     </gazebo>
-    <gazebo reference="joint_chassis_right_rear_wheel">
+    <gazebo reference="camera_joint">
         <preserveFixedJoint>true</preserveFixedJoint>
-    </gazebo>  -->
+    </gazebo>
+    <gazebo reference="left_wheel">
+        <kp>1000000000000000000000000000.0</kp>
+        <kd>1000000000000000000000000000.0</kd>
+        <mu1>10.0</mu1>
+        <mu2>10.0</mu2>
+        <material>Gazebo/Orange</material>
+    </gazebo>
+    <gazebo reference="right_wheel">
+        <kp>1000000000000000000000000000.0</kp>
+        <kd>1000000000000000000000000000.0</kd>
+        <mu1>10.0</mu1>
+        <mu2>10.0</mu2>
+        <material>Gazebo/Orange</material>
+    </gazebo>
+    <!-- JOINT PUBLISHER -->
+    <gazebo>
+        <plugin name="ros_tank_joint_state" filename="libgazebo_ros_joint_state_publisher.so">
+            <ros>
+                <remapping>~/out:=joint_states</remapping>
+            </ros>
+            <update_rate>30</update_rate>
+            <joint_name>camera_servo_first_joint</joint_name>
+            <joint_name>camera_servo_second_joint</joint_name>
+            <joint_name>joint_left_wheel</joint_name>
+            <joint_name>joint_right_wheel</joint_name>
+        </plugin>
+    </gazebo>
+    <!-- Differential drive -->
+    <gazebo>
+        <plugin filename="libgazebo_ros_diff_drive.so" name="differential_drive_controller">
+            <!-- wheels -->
+            <left_joint>joint_left_wheel</left_joint>
+            <right_joint>joint_right_wheel</right_joint>
+            <!-- kinematics -->
+            <wheel_separation>0.1</wheel_separation>
+            <wheel_diameter>0.04</wheel_diameter>
+            <!-- limits -->
+            <max_wheel_torque>1.0</max_wheel_torque>
+            <max_wheel_acceleration>2.0</max_wheel_acceleration>
+            <!-- output -->
+            <publish_odom>true</publish_odom>
+            <publish_odom_tf>true</publish_odom_tf>
+            <odometry_frame>odom</odometry_frame>
+            <robot_base_frame>base_link</robot_base_frame>
+        </plugin>
+    </gazebo>
+    <!-- Pointcloud plugin -->
+    <gazebo reference="pointcloud_link">
+        <sensor type="ray" name="pointcloud_sensor">
+            <ray>
+            <scan>
+                <horizontal>
+                    <samples>50</samples>
+                    <resolution>1.0</resolution>
+                    <min_angle>-1.0</min_angle>
+                    <max_angle>1.0</max_angle>
+                </horizontal>
+                <vertical>
+                    <samples>50</samples>
+                    <resolution>1.0</resolution>
+                    <min_angle>-1.0</min_angle>
+                    <max_angle>1.0</max_angle>
+                </vertical>
+            </scan>
+            <range>
+                <min>0.10</min>
+                <max>5.0</max>
+                <resolution>0.01</resolution>
+            </range>
+            <!-- Using gazebo's noise instead of plugin's -->
+            <noise>
+                <type>gaussian</type>
+                <mean>0.0</mean>
+                <stddev>0.01</stddev>
+            </noise>
+            </ray>
+            <!-- Using gazebo's update rate instead of plugin's -->
+            <update_rate>30</update_rate>
+            <plugin name="gazebo_ros_block_laser_controller" filename="libgazebo_ros_ray_sensor.so">
+            <!-- Change namespace and output topic so published topic is /rrbot/laser/pointcloud -->
+            <ros>
+                <namespace>box_bot</namespace>
+                <argument>~/out:=pointcloud</argument>
+            </ros>
+            <!-- Set output to sensor_msgs/PointCloud to get same output type as gazebo_ros_block_laser -->
+            <output_type>sensor_msgs/PointCloud</output_type>
+            <frame_name>pointcloud_link</frame_name>
+            <!-- min_intensity instead of hokuyoMinIntensity -->
+            <min_intensity>100.0</min_intensity>
+            </plugin>
+        </sensor>
+    </gazebo>
+    <!-- Camera plugin -->
+     <gazebo reference="camera_link">
+        <sensor name="camera_robot" type="camera">
+            <camera>
+                <pose> 0 0 0 0 0 0 </pose>
+                <visualize>true</visualize>
+                <update_rate>10</update_rate>
+                <horizontal_fov>1.089</horizontal_fov>
+                <image>
+                    <format>R8G8B8</format>
+                    <width>640</width>
+                    <height>480</height>
+                </image>
+                <noise>
+                    <type>gaussian</type>
+                    <mean>0.0</mean>
+                    <stddev>0.007</stddev>
+                </noise>
+            </camera>
+            <plugin name="camera_controller" filename="libgazebo_ros_camera.so">
+                <alwaysOn>true</alwaysOn>
+                <updateRate>0.0</updateRate>
+                <imageTopicName>image_raw</imageTopicName>
+                <cameraName>camera</cameraName>
+                <cameraInfoTopicName>camera_info</cameraInfoTopicName>
+                <frameName>link_chassis</frameName>
+            </plugin>
+        </sensor>
+    </gazebo>
+    <!-- Laser scan plugin -->
     <gazebo reference="link_laser_scan">
         <sensor type="ray" name="head_hokuyo_sensor">
             <pose>0 0 0 0 0 0</pose>
-            <visualize>true</visualize>
+            <always_on>true</always_on>
+            <visualize>false</visualize>
             <update_rate>20</update_rate>
             <ray>
@@ -36,32 +176,12 @@
                 </noise>
             </ray>
-            <plugin name="gazebo_ros_head_hokuyo_controller" filename="libgazebo_ros_laser.so">
-                <topicName>/laser/scan</topicName>
-                <frameName>link_chassis</frameName>
+            <plugin name="laser" filename="libgazebo_ros_ray_sensor.so">
+                <ros>
+                    <namespace>/ros_tank</namespace>
+                    <remapping>~/out:=laser_scan</remapping>
+                </ros>
+                <output_type>sensor_msgs/LaserScan</output_type>
             </plugin>
         </sensor>
     </gazebo>
-<!--
-    <gazebo>
-        <plugin filename="libgazebo_ros_diff_drive.so" name="differential_drive_controller">
-            <alwaysOn>true</alwaysOn>
-            <updateRate>20</updateRate>
-            <leftJoint>joint_chassis_left_middle_wheel</leftJoint>
-            <rightJoint>joint_chassis_right_middle_wheel</rightJoint>
-            <wheelSeparation>0.14</wheelSeparation>
-            <wheelDiameter>0.04</wheelDiameter>
-            <torque>10</torque>
-            <wheelTorque>5</wheelTorque>
-            <commandTopic>cmd_vel</commandTopic>
-            <odometryTopic>odom</odometryTopic>
-            <odometryFrame>odom</odometryFrame>
-            <robotBaseFrame>link_chassis</robotBaseFrame>
-            <publishWheelTF>false</publishWheelTF>
-            <publishWheelJointState>false</publishWheelJointState>
-            <publishOdomTF>true</publishOdomTF>
-            <wheelAcceleration>0</wheelAcceleration>
-            <rosDebugLevel>na</rosDebugLevel>
-            <odometrySource>world</odometrySource>
-            <publishTf>1</publishTf>
-        </plugin>
-    </gazebo> -->
+</robot>
