Commit message: Added gazebo.xacro

File: ros_tank_description/urdf/robot.xacro (robot description, xacro)
@@ -1,158 +1,8 @@
-<?xml version="1.0"?>
-<robot name="ros_tank">
-    <gazebo reference="joint_laser_scan_chassis">
-        <preserveFixedJoint>true</preserveFixedJoint>
-    </gazebo>
-    <gazebo reference="camera_servo_first_joint">
-        <preserveFixedJoint>true</preserveFixedJoint>
-    </gazebo>
-    <gazebo reference="camera_servo_second_joint">
-        <preserveFixedJoint>true</preserveFixedJoint>
-    </gazebo>
-    <gazebo reference="camera_joint">
-        <preserveFixedJoint>true</preserveFixedJoint>
-    </gazebo>
-    <gazebo reference="link_laser_scan">
-        <material>Gazebo/Red</material>
-    </gazebo>
-    <gazebo reference="link_chassis">
-        <material>Gazebo/DarkGrey</material>
-    </gazebo>
-    <gazebo reference="camera_servo_first_link">
-        <material>Gazebo/Red</material>
-    </gazebo>
-    <gazebo reference="camera_link">
-        <material>Gazebo/Red</material>
-    </gazebo>
-    <gazebo reference="camera_second_servo_link">
-        <material>Gazebo/Blue</material>
-    </gazebo>
-    <!-- JOINT PUBLISHER -->
-    <gazebo>
-        <plugin name="ros_tank_joint_state" filename="libgazebo_ros_joint_state_publisher.so">
-            <ros>
-                <remapping>~/out:=joint_states</remapping>
-            </ros>
-            <update_rate>30</update_rate>
-            <joint_name>camera_servo_first_joint</joint_name>
-            <joint_name>camera_servo_second_joint</joint_name>
-            <joint_name>joint_chassis_left_middle_wheel</joint_name>
-            <joint_name>joint_chassis_right_middle_wheel</joint_name>
-        </plugin>
-    </gazebo>
-     <gazebo reference="camera_link">
-        <sensor name="camera_robot" type="camera">
-            <camera>
-                <pose> 0 0 0 0 0 0 </pose>
-                <visualize>true</visualize>
-                <update_rate>10</update_rate>
-                <horizontal_fov>1.089</horizontal_fov>
-                <image>
-                    <format>R8G8B8</format>
-                    <width>640</width>
-                    <height>480</height>
-                </image>
-                <noise>
-                    <type>gaussian</type>
-                    <mean>0.0</mean>
-                    <stddev>0.007</stddev>
-                </noise>
-            </camera>
-            <plugin name="camera_controller" filename="libgazebo_ros_camera.so">
-                <alwaysOn>true</alwaysOn>
-                <updateRate>0.0</updateRate>
-                <imageTopicName>image_raw</imageTopicName>
-                <cameraName>camera</cameraName>
-                <cameraInfoTopicName>camera_info</cameraInfoTopicName>
-                <frameName>link_chassis</frameName>
-            </plugin>
-        </sensor>
-    </gazebo>
-    <gazebo reference="link_laser_scan">
-        <sensor type="ray" name="head_hokuyo_sensor">
-            <pose>0 0 0 0 0 0</pose>
-            <always_on>true</always_on>
-            <visualize>true</visualize>
-            <update_rate>20</update_rate>
-            <ray>
-                <scan>
-                    <horizontal>
-                        <samples>720</samples>
-                        <resolution>1</resolution>
-                        <min_angle>-3.14</min_angle>
-                        <max_angle>3.14</max_angle>
-                    </horizontal>
-                </scan>
-                <range>
-                    <min>0.20</min>
-                    <max>12.0</max>
-                    <resolution>0.01</resolution>
-                </range>
-                <noise>
-                    <type>gaussian</type>
-                    <mean>0.0</mean>
-                    <stddev>0.01</stddev>
-                </noise>
-            </ray>
-            <plugin name="laser" filename="libgazebo_ros_ray_sensor.so">
-                <ros>
-                    <namespace>/ros_tank</namespace>
-                    <remapping>~/out:=laser_scan</remapping>
-                </ros>
-                <output_type>sensor_msgs/LaserScan</output_type>
-            </plugin>
-        </sensor>
-    </gazebo>
-    <gazebo reference="link_front_left_wheel">
-        <material>Gazebo/Black</material>
-        <kp>1000000000000000000000000000.0</kp>
-        <kd>1000000000000000000000000000.0</kd>
-        <mu1>0.01</mu1>
-        <mu2>0.01</mu2>
-    </gazebo>
-    <gazebo reference="link_rear_right_wheel">
-        <material>Gazebo/Black</material>
-        <kp>1000000000000000000000000000.0</kp>
-        <kd>1000000000000000000000000000.0</kd>
-        <mu1>0.01</mu1>
-        <mu2>0.01</mu2>
-    </gazebo>
-    <gazebo reference="link_rear_left_wheel">
-        <material>Gazebo/Black</material>
-        <kp>1000000000000000000000000000.0</kp>
-        <kd>1000000000000000000000000000.0</kd>
-        <mu1>0.01</mu1>
-        <mu2>0.01</mu2>
-    </gazebo>
-    <gazebo reference="link_front_right_wheel">
-        <material>Gazebo/Black</material>
-        <kp>1000000000000000000000000000.0</kp>
-        <kd>1000000000000000000000000000.0</kd>
-        <mu1>0.01</mu1>
-        <mu2>0.01</mu2>
-    </gazebo>
-    <gazebo reference="link_middle_right_wheel">
-        <material>Gazebo/Black</material>
-        <kp>1000000000000000000000000000.0</kp>
-        <kd>1000000000000000000000000000.0</kd>
-        <mu1>10</mu1>
-        <mu2>10</mu2>
-    </gazebo>
-    <gazebo reference="link_middle_left_wheel">
-        <material>Gazebo/Black</material>
-        <kp>1000000000000000000000000000.0</kp>
-        <kd>1000000000000000000000000000.0</kd>
-        <mu1>10</mu1>
-        <mu2>10</mu2>
-    </gazebo>
+<?xml version="1.0" ?>
+<robot name="ros_tank" xmlns:xacro="http://www.ros.org/wiki/xacro">
+    <xacro:include filename="$(find ros_tank_description)/urdf/gazebo.xacro" />
     <link name="base_link"></link>
     <!-- Link - chassis -->
     <link name="link_chassis">
-        <collision>
-            <origin xyz="0 0 -0.08" rpy="0 0 0"/>
-            <geometry>
-                <box size="0.25 0.25 0.1" />
-            </geometry>
-        </collision>
         <visual>
             <geometry>
@@ -164,4 +14,10 @@
             </material>
         </visual>
+        <collision>
+            <origin xyz="0 0 -0.08" rpy="0 0 0"/>
+            <geometry>
+                <box size="0.25 0.25 0.1" />
+            </geometry>
+        </collision>
         <inertial>
             <mass value="0.5"/>
@@ -175,209 +31,5 @@
         <child link="link_chassis" />
     </joint>
-    <!-- Link - left front wheel -->
-    <link name="link_front_left_wheel">
-        <inertial>
-            <mass value="10" />
-            <origin xyz="0 0 0.3" rpy="0 0 0" />
-            <inertia ixx="1.5417" ixy="0" ixz="0" iyy="3.467" iyz="0" izz="4.742" />
-        </inertial>
-        <collision>
-            <origin rpy="1.5707 0 0" xyz="0 -0.015 0" />
-            <geometry>
-                <cylinder length="0.03" radius="0.02"/>
-            </geometry>
-        </collision>
-        <visual>
-            <origin rpy="1.5707 0 0" xyz="0 0.015 0" />
-            <geometry>
-                <cylinder length="0.03" radius="0.02"/>
-            </geometry>
-        </visual>
-        <inertial>
-            <origin rpy="0 1.5707 1.5707" xyz="0 0 0"/>
-            <mass value="0.01"/>
-            <inertia ixx="5.145833333333334e-09" ixy="0" ixz="0" iyy="5.145833333333334e-09" iyz="0" izz="1.0125000000000003e-08"/>
-        </inertial>
-    </link>
-    <!-- Joint - chassis / left front wheel -->
-    <joint name="joint_chassis_left_front_wheel" type="fixed">
-        <origin rpy="0 0 0" xyz="0.065 0.077 -0.12" />
-        <child link="link_front_left_wheel" />
-        <parent link="link_chassis" />
-        <axis rpy="0 0 0" xyz="0 1 0" />
-        <limit effort="10000" velocity="1000" />
-        <joint_properties damping="1.0" friction="1.0" />
-    </joint>
-    <!-- Link - left middle wheel -->
-    <link name="link_middle_left_wheel">
-        <inertial>
-            <mass value="10" />
-            <origin xyz="0 0 0.3" rpy="0 0 0" />
-            <inertia ixx="1.5417" ixy="0" ixz="0" iyy="3.467" iyz="0" izz="4.742" />
-        </inertial>
-        <collision>
-            <origin rpy="1.5707 0 0" xyz="0 0.015 0" />
-            <geometry>
-                <cylinder length="0.03" radius="0.02"/>
-            </geometry>
-        </collision>
-        <visual>
-            <origin rpy="1.5707 0 0" xyz="0 0.015 0" />
-            <geometry>
-                <cylinder length="0.03" radius="0.02"/>
-            </geometry>
-        </visual>
-        <inertial>
-            <origin rpy="0 1.5707 1.5707" xyz="0 0 0"/>
-            <mass value="0.01"/>
-            <inertia ixx="5.145833333333334e-09" ixy="0" ixz="0" iyy="5.145833333333334e-09" iyz="0" izz="1.0125000000000003e-08"/>
-        </inertial>
-    </link>
-    <!-- Joint - chassis / left middle wheel -->
-    <joint name="joint_chassis_left_middle_wheel" type="continuous">
-        <origin rpy="0 0 0" xyz="0 0.077 -0.12" />
-        <child link="link_middle_left_wheel" />
-        <parent link="link_chassis" />
-        <axis rpy="0 0 0" xyz="0 1 0" />
-        <limit effort="10000" velocity="1000" />
-        <joint_properties damping="1.0" friction="1.0" />
-    </joint>
-    <!-- Link - left rear wheel -->
-    <link name="link_rear_left_wheel">
-        <inertial>
-            <mass value="10" />
-            <origin xyz="0 0 0.3" rpy="0 0 0" />
-            <inertia ixx="1.5417" ixy="0" ixz="0" iyy="3.467" iyz="0" izz="4.742" />
-        </inertial>
-        <collision>
-            <origin rpy="1.5707 0 0" xyz="0 0.015 0" />
-            <geometry>
-                <cylinder length="0.03" radius="0.02"/>
-            </geometry>
-        </collision>
-        <visual>
-            <origin rpy="1.5707 0 0" xyz="0 0.015 0" />
-            <geometry>
-                <cylinder length="0.03" radius="0.02"/>
-            </geometry>
-        </visual>
-        <inertial>
-            <origin rpy="0 1.5707 1.5707" xyz="0 0 0"/>
-            <mass value="0.01"/>
-            <inertia ixx="5.145833333333334e-09" ixy="0" ixz="0" iyy="5.145833333333334e-09" iyz="0" izz="1.0125000000000003e-08"/>
-        </inertial>
-    </link>
-    <!-- Joint - chassis / left rear wheel -->
-    <joint name="joint_chassis_left_rear_wheel" type="fixed">
-        <origin rpy="0 0 0" xyz="-0.065 0.077 -0.12" />
-        <child link="link_rear_left_wheel" />
-        <parent link="link_chassis" />
-        <axis rpy="0 0 0" xyz="0 1 0" />
-        <limit effort="10000" velocity="1000" />
-        <joint_properties damping="1.0" friction="1.0" />
-    </joint>
-    <!-- Joint - chassis / right front wheel -->
-    <joint name="joint_chassis_right_front_wheel" type="fixed">
-        <origin rpy="0 0 0" xyz="0.065 -0.077 -0.12" />
-        <child link="link_front_right_wheel" />
-        <parent link="link_chassis" />
-        <axis rpy="0 0 0" xyz="0 1 0" />
-        <limit effort="10000" velocity="1000" />
-        <joint_properties damping="1.0" friction="1.0" />
-    </joint>
-    <!-- Link - right front wheel -->
-    <link name="link_front_right_wheel">
-        <inertial>
-            <mass value="10" />
-            <origin xyz="0 0 0.3" rpy="0 0 0" />
-            <inertia ixx="1.5417" ixy="0" ixz="0" iyy="3.467" iyz="0" izz="4.742" />
-        </inertial>
-        <collision>
-            <origin rpy="1.5707 0 0" xyz="0 -0.015 0" />
-            <geometry>
-                <cylinder length="0.03" radius="0.02"/>
-            </geometry>
-        </collision>
-        <visual>
-            <origin rpy="1.5707 0 0" xyz="0 -0.015 0" />
-            <geometry>
-                <cylinder length="0.03" radius="0.02"/>
-            </geometry>
-        </visual>
-        <inertial>
-            <origin rpy="0 1.5707 1.5707" xyz="0 0 0"/>
-            <mass value="0.01"/>
-            <inertia ixx="5.145833333333334e-09" ixy="0" ixz="0" iyy="5.145833333333334e-09" iyz="0" izz="1.0125000000000003e-08"/>
-        </inertial>
-    </link>
-    <!-- Joint - chassis / right middle wheel -->
-    <joint name="joint_chassis_right_middle_wheel" type="continuous">
-        <origin rpy="0 0 0" xyz="0 -0.077 -0.12" />
-        <child link="link_middle_right_wheel" />
-        <parent link="link_chassis" />
-        <axis rpy="0 0 0" xyz="0 1 0" />
-        <limit effort="10000" velocity="1000" />
-        <joint_properties damping="1.0" friction="1.0" />
-    </joint>
-    <!-- Link - right middle wheel -->
-    <link name="link_middle_right_wheel">
-        <inertial>
-            <mass value="10" />
-            <origin xyz="0 0 0.3" rpy="0 0 0" />
-            <inertia ixx="1.5417" ixy="0" ixz="0" iyy="3.467" iyz="0" izz="4.742" />
-        </inertial>
-        <collision>
-            <origin rpy="1.5707 0 0" xyz="0 -0.015 0" />
-            <geometry>
-                <cylinder length="0.03" radius="0.02"/>
-            </geometry>
-        </collision>
-        <visual>
-            <origin rpy="1.5707 0 0" xyz="0 -0.015 0" />
-            <geometry>
-                <cylinder length="0.03" radius="0.02"/>
-            </geometry>
-        </visual>
-        <inertial>
-            <origin rpy="0 1.5707 1.5707" xyz="0 0 0"/>
-            <mass value="0.01"/>
-            <inertia ixx="5.145833333333334e-09" ixy="0" ixz="0" iyy="5.145833333333334e-09" iyz="0" izz="1.0125000000000003e-08"/>
-        </inertial>
-    </link>
-     <!-- Joint - chassis / right rear wheel -->
-    <joint name="joint_chassis_right_rear_wheel" type="fixed">
-        <origin rpy="0 0 0" xyz="-0.065 -0.077 -0.12" />
-        <child link="link_rear_right_wheel" />
-        <parent link="link_chassis" />
-        <axis rpy="0 0 0" xyz="0 1 0" />
-        <limit effort="10000" velocity="1000" />
-        <joint_properties damping="1.0" friction="1.0" />
-    </joint>
-    <!-- Link - right rear wheel -->
-    <link name="link_rear_right_wheel">
-        <inertial>
-            <mass value="10" />
-            <origin xyz="0 0 0.3" rpy="0 0 0" />
-            <inertia ixx="1.5417" ixy="0" ixz="0" iyy="3.467" iyz="0" izz="4.742" />
-        </inertial>
-        <collision>
-            <origin rpy="1.5707 0 0" xyz="0 -0.015 0" />
-            <geometry>
-                <cylinder length="0.03" radius="0.02"/>
-            </geometry>
-        </collision>
-        <visual>
-            <origin rpy="1.5707 0 0" xyz="0 -0.015 0" />
-            <geometry>
-                <cylinder length="0.03" radius="0.02"/>
-            </geometry>
-        </visual>
-        <inertial>
-            <origin rpy="0 1.5707 1.5707" xyz="0 0 0"/>
-            <mass value="0.01"/>
-            <inertia ixx="5.145833333333334e-09" ixy="0" ixz="0" iyy="5.145833333333334e-09" iyz="0" izz="1.0125000000000003e-08"/>
-        </inertial>
-    </link>
-    <!-- Laser scan -->
+    <!-- Joint - laser scan -->
     <joint name="joint_laser_scan_chassis" type="fixed">
         <origin rpy="0 0 0" xyz="-0.01 0 0.11" />
@@ -386,10 +38,6 @@
         <joint_properties damping="1.0" friction="1.0" />
     </joint>
+    <!-- Link - laser scan -->
     <link name="link_laser_scan">
-        <inertial>
-            <origin xyz="0 0 0" rpy="0 0 0" />
-            <mass value="0.5" />
-            <inertia ixx="0.000252666666667" ixy="0" ixz="0" iyy="0.000252666666667" iyz="0" izz="0.0005"/>
-        </inertial>
         <visual>
             <origin xyz="0 0 0" rpy="0 0 0" />
@@ -423,14 +71,8 @@
     </joint>
     <!-- Link - camera second servo -->
-     <link name="camera_second_servo_link">
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