Commit message: Added controllers to the robot

File: ros_tank_description/urdf/robot.xacro (robot description, xacro)
@@ -2,4 +2,5 @@
 <robot name="ros_tank" xmlns:xacro="http://www.ros.org/wiki/xacro">
     <xacro:include filename="$(find ros_tank_description)/urdf/gazebo.xacro" />
+    <xacro:include filename="$(find ros_tank_description)/urdf/control.xacro" />
     <link name="base_link"></link>
     <!-- Link - chassis -->
@@ -78,5 +79,5 @@
                 <mesh filename="package://ros_tank_description/meshes/camera_servo_2.stl" pose="0 0 0" scale="0.0011 0.00111 0.0011"/>
             </geometry>
-            <material name="Gazebo/DarkGrey" />
+            <!-- <material name="Gazebo/DarkGrey" /> -->
         </visual>
         <collision>
@@ -108,5 +109,5 @@
                 <!-- <box size="0.03 0.04 0.05" /> -->
             </geometry>
-            <material name="Gazebo/Orange" />
+            <!-- <material name="Gazebo/Orange" /> -->
         </visual>
         <collision>
@@ -173,5 +174,4 @@
             <cylinder length="0.001" radius="0.015"/>
             </geometry>
-            <material name="red"/>
         </visual>
         <collision>
@@ -203,5 +203,4 @@
             <cylinder length="0.001" radius="0.015"/>
             </geometry>
-            <material name="green"/>
         </visual>
         <collision>
