Commit message: Refactored code

File: ros_tank_description/urdf/control.xacro (robot description, xacro)
@@ -1,5 +1,5 @@
 <?xml version="1.0"?>
 <robot>
-    <ros2_control name="MyRobotSystem" type="system">
+    <ros2_control name="camera_controller" type="system">
         <hardware>
             <plugin>gazebo_ros2_control/GazeboSystem</plugin>
@@ -20,10 +20,26 @@
         </joint>
     </ros2_control>
-    <!-- Gazebo's ros2_control plugin -->
-    <gazebo>
-    <plugin filename="libgazebo_ros2_control.so" name="gazebo_ros2_control">
-        <robot_sim_type>gazebo_ros2_control/GazeboSystem</robot_sim_type>
-        <parameters>$(find ros_tank_control)/config/ros_tank_controllers.yaml</parameters>
-    </plugin>
-    </gazebo>
+    <ros2_control name="diff_drive" type="system">
+      <hardware>
+          <plugin>gazebo_ros2_control/GazeboSystem</plugin>
+      </hardware>
+      <joint name="joint_left_wheel">
+        <command_interface name="velocity">
+          <param name="min">-1</param>
+          <param name="max">1</param>
+        </command_interface>
+        <state_interface name="position"/>
+        <state_interface name="velocity"/>
+        <state_interface name="effort"/>
+      </joint>
+      <joint name="joint_right_wheel">
+        <command_interface name="velocity">
+          <param name="min">-1</param>
+          <param name="max">1</param>
+        </command_interface>
+        <state_interface name="position"/>
+        <state_interface name="velocity"/>
+        <state_interface name="effort"/>
+      </joint>
+    </ros2_control>
 </robot>

File: ros_tank_description/urdf/gazebo.xacro (robot description, xacro)
@@ -43,5 +43,5 @@
     </gazebo>
     <!-- JOINT PUBLISHER -->
-    <gazebo>
+    <!-- <gazebo>
         <plugin name="ros_tank_joint_state" filename="libgazebo_ros_joint_state_publisher.so">
             <ros>
@@ -54,5 +54,5 @@
             <joint_name>joint_right_wheel</joint_name>
         </plugin>
-    </gazebo>
+    </gazebo> -->
     <!-- Differential drive -->
     <gazebo>
@@ -74,4 +74,11 @@
         </plugin>
     </gazebo>
+    <!-- Gazebo's ros2_control plugin -->
+    <!-- <gazebo>
+        <plugin filename="libgazebo_ros2_control.so" name="gazebo_ros2_control">
+            <robot_sim_type>gazebo_ros2_control/GazeboSystem</robot_sim_type>
+            <parameters>$(find ros_tank_control)/config/ros_tank_controllers.yaml</parameters>
+        </plugin>
+    </gazebo> -->
     <!-- Pointcloud plugin -->
     <gazebo reference="pointcloud_link">

File: ros_tank_description/urdf/robot_sim.xacro (robot description, xacro)
@@ -2,4 +2,4 @@
 <robot name="ros_tank" xmlns:xacro="http://www.ros.org/wiki/xacro">
     <xacro:include filename="$(find ros_tank_description)/urdf/base_urdf.xacro" />
-    <xacro:include filename="$(find ros_tank_description)/urdf/control_real.xacro" />
+    <xacro:include filename="$(find ros_tank_description)/urdf/gazebo.xacro" />
 </robot>
