Commit message: Updated urdf file

File: ros_tank_description/urdf/base_urdf.xacro (robot description, xacro)
@@ -20,7 +20,7 @@
         </collision>
         <inertial>
-            <mass value="0.5"/>
+            <mass value="10"/>
             <origin rpy="0 0 0" xyz="0 0 0"/>
-            <inertia ixx="0.0008333333333333335" ixy="0" ixz="0" iyy="0.0008333333333333335" iyz="0" izz="0.0008333333333333335"/>
+            <inertia ixx="0.1" ixy="0" ixz="0" iyy="0.1" iyz="0" izz="0.1"/>
         </inertial>
     </link>
@@ -56,7 +56,7 @@
         </collision>
         <inertial>
-            <mass value="0.01"/>
+            <mass value="0.1"/>
             <origin rpy="0 0 0" xyz="0 0 0.0204"/>
-            <inertia ixx="6.066578520833334e-06" ixy="0" ixz="0" iyy="6.072950163333333e-06" iyz="0" izz="9.365128684166666e-06"/>
+            <inertia ixx="0.01" ixy="0.0" ixz="0.0" iyy="0.01" iyz="0.0" izz="0.01"/>
         </inertial>
     </link>
@@ -67,5 +67,5 @@
         <child link="camera_second_servo_link"/>
         <axis xyz="0 1 0"/>
-        <limit lower="-1.15" upper="1.4" velocity="100" effort="100"/>
+        <limit lower="-1.15" upper="1.4" velocity="1" effort="5"/>
     </joint>
     <!-- Link - camera second servo -->
@@ -77,5 +77,5 @@
                 <mesh filename="package://ros_tank_description/meshes/camera_servo_2.stl" pose="0 0 0" scale="0.0011 0.00111 0.0011"/>
             </geometry>
-            <!-- <material name="Gazebo/DarkGrey" /> -->
+            <material name="Gazebo/DarkGrey" />
         </visual>
         <collision>
@@ -86,7 +86,7 @@
         </collision>
         <inertial>
-            <mass value="0.01"/>
-            <origin rpy="0 0 0" xyz="0 0 0.0204"/>
-            <inertia ixx="6.066578520833334e-06" ixy="0" ixz="0" iyy="6.072950163333333e-06" iyz="0" izz="9.365128684166666e-06"/>
+            <mass value="0.1"/>
+            <origin rpy="0 0 0" xyz="0 0 0"/>
+            <inertia ixx="0.1" ixy="0.0" ixz="0.0" iyy="0.1" iyz="0.0" izz="0.1"/>
         </inertial>
     </link>
@@ -97,5 +97,5 @@
         <child link="camera_servo_first_link"/>
         <axis xyz="0 0 1"/>
-        <limit lower="-1.15" upper="1.4" velocity="100" effort="100"/>
+        <limit lower="-1.15" upper="1.4" velocity="1" effort="5"/>
     </joint>
     <!-- Link - camera first servo -->
@@ -116,7 +116,7 @@
         </collision>
         <inertial>
-            <mass value="0.01"/>
-            <origin rpy="0 0 0" xyz="0 0 0.0204"/>
-            <inertia ixx="6.066578520833334e-06" ixy="0" ixz="0" iyy="6.072950163333333e-06" iyz="0" izz="9.365128684166666e-06"/>
+            <mass value="0.1"/>
+            <origin rpy="0 0 0" xyz="0 0 0"/>
+            <inertia ixx="0.1" ixy="0.0" ixz="0.0" iyy="0.1" iyz="0.0" izz="0.1"/>
         </inertial>
     </link>
@@ -142,5 +142,5 @@
         </collision>
         <inertial>
-            <mass value="0.003"/>
+            <mass value="0.1"/>
             <origin rpy="0 0 0" xyz="0 0 0.0204"/>
             <inertia ixx="6.066578520833334e-06" ixy="0" ixz="0" iyy="6.072950163333333e-06" iyz="0" izz="9.365128684166666e-06"/>

Commit message: Added second Dokerfile

File: ros_tank_description/urdf/base_urdf.xacro (robot description, xacro)
@@ -59,90 +59,4 @@
             <origin rpy="0 0 0" xyz="0 0 0.0204"/>
             <inertia ixx="0.01" ixy="0.0" ixz="0.0" iyy="0.01" iyz="0.0" izz="0.01"/>
-        </inertial>
-    </link>
-     <!-- Joint - camera second servo -->
-    <joint name="camera_servo_second_joint" type="revolute">
-        <origin xyz="0.03 -0.005 0.02" rpy="0 0 0"/>
-        <parent link="camera_servo_first_link"/>
-        <child link="camera_second_servo_link"/>
-        <axis xyz="0 1 0"/>
-        <limit lower="-1.15" upper="1.4" velocity="1" effort="5"/>
-    </joint>
-    <!-- Link - camera second servo -->
-    <link name="camera_second_servo_link">
-        <visual>
-            <origin xyz="0 0 0" rpy="0 0 0"/>
-            <geometry>
-                <!-- <box size="0.02 0.03 0.03" /> -->
-                <mesh filename="package://ros_tank_description/meshes/camera_servo_2.stl" pose="0 0 0" scale="0.0011 0.00111 0.0011"/>
-            </geometry>
-            <material name="Gazebo/DarkGrey" />
-        </visual>
-        <collision>
-            <origin xyz="0 0 0.01" rpy="0 0 0"/>
-            <geometry>
-                <box size="0.02 0.03 0.03" />
-            </geometry>
-        </collision>
-        <inertial>
-            <mass value="0.1"/>
-            <origin rpy="0 0 0" xyz="0 0 0"/>
-            <inertia ixx="0.1" ixy="0.0" ixz="0.0" iyy="0.1" iyz="0.0" izz="0.1"/>
-        </inertial>
-    </link>
-     <!-- Joint - camera first servo -->
-    <joint name="camera_servo_first_joint" type="revolute">
-        <origin xyz="0.053 0 0" rpy="0 0 0"/>
-        <parent link="link_chassis"/>
-        <child link="camera_servo_first_link"/>
-        <axis xyz="0 0 1"/>
-        <limit lower="-1.15" upper="1.4" velocity="1" effort="5"/>
-    </joint>
-    <!-- Link - camera first servo -->
-    <link name="camera_servo_first_link">
-        <visual>
-            <origin xyz="0 0 0" rpy="0 0 0"/>
-            <geometry>
-                <mesh filename="package://ros_tank_description/meshes/camera_servo_1.stl" pose="0 0 0" scale="0.0011 0.00111 0.0011"/>
-                <!-- <box size="0.03 0.04 0.05" /> -->
-            </geometry>
-            <!-- <material name="Gazebo/Orange" /> -->
-        </visual>
-        <collision>
-            <origin xyz="0 0 -0.005" rpy="0 0 0"/>
-            <geometry>
-                <box size="0.03 0.04 0.03" />
-            </geometry>
-        </collision>
-        <inertial>
-            <mass value="0.1"/>
-            <origin rpy="0 0 0" xyz="0 0 0"/>
-            <inertia ixx="0.1" ixy="0.0" ixz="0.0" iyy="0.1" iyz="0.0" izz="0.1"/>
-        </inertial>
-    </link>
-    <!-- Joint - camera -->
-    <joint name="camera_joint" type="fixed">
-        <parent link="camera_second_servo_link"/>
-        <child link="camera_link"/>
-        <origin xyz="0.03 0 0.017" rpy="0 0 0"/>
-    </joint>
-    <!-- Link - camera -->
-    <link name="camera_link">
-        <visual>
-            <geometry>
-                <mesh filename="package://ros_tank_description/meshes/camera.stl" pose="0 0 0" scale="0.00111 0.00111 0.0011"/>
-                <!-- <box size="0.02 0.08 0.038"/> -->
-            </geometry>
-        </visual>
-        <collision>
-            <origin xyz="0 0 0" rpy="0 0 0"/>
-            <geometry>
-                <box size="0.02 0.08 0.038"/>
-            </geometry>
-        </collision>
-        <inertial>
-            <mass value="0.1"/>
-            <origin rpy="0 0 0" xyz="0 0 0.0204"/>
-            <inertia ixx="6.066578520833334e-06" ixy="0" ixz="0" iyy="6.072950163333333e-06" iyz="0" izz="9.365128684166666e-06"/>
         </inertial>
     </link>

File: ros_tank_description/urdf/control.xacro (robot description, xacro)
@@ -20,27 +20,4 @@
         </joint>
     </ros2_control>
-    <!-- <ros2_control name="diff_drive" type="system">
-      <hardware>
-          <plugin>gazebo_ros2_control/GazeboSystem</plugin>
-      </hardware>
-      <joint name="joint_left_wheel">
-        <command_interface name="velocity">
-          <param name="min">-1</param>
-          <param name="max">1</param>
-        </command_interface>
-        <state_interface name="position"/>
-        <state_interface name="velocity"/>
-        <state_interface name="effort"/>
-      </joint>
-      <joint name="joint_right_wheel">
-        <command_interface name="velocity">
-          <param name="min">-1</param>
-          <param name="max">1</param>
-        </command_interface>
-        <state_interface name="position"/>
-        <state_interface name="velocity"/>
-        <state_interface name="effort"/>
-      </joint>
-    </ros2_control> -->
     <!-- Gazebo's ros2_control plugin -->
     <gazebo>

File: ros_tank_description/urdf/robot.xacro (robot description, xacro)
@@ -2,4 +2,4 @@
 <robot name="ros_tank" xmlns:xacro="http://www.ros.org/wiki/xacro">
     <xacro:include filename="$(find ros_tank_description)/urdf/base_urdf.xacro" />
-    <xacro:include filename="$(find ros_tank_description)/urdf/control.xacro" />
+    <xacro:include filename="$(find ros_tank_description)/urdf/control_arduino.xacro" />
 </robot>
