Commit message: Added  camera and lidar nodes

File: ros2_ws/ros_tank_description/urdf/base_urdf.xacro (robot description, xacro)
@@ -32,5 +32,5 @@
     <!-- Joint - laser scan -->
     <joint name="joint_laser_scan_chassis" type="fixed">
-        <origin rpy="0 0 0" xyz="-0.01 0 0.11" />
+        <origin rpy="0 0 3.2" xyz="-0.01 0 0.11" />
         <child link="link_laser_scan" />
         <parent link="link_chassis" />

Commit message: Added camera joints

File: ros2_ws/ros_tank_description/urdf/base_urdf.xacro (robot description, xacro)
@@ -40,5 +40,5 @@
     <link name="link_laser_scan">
         <visual>
-            <origin xyz="0 0 0" rpy="0 0 0" />
+            <origin xyz="0 0 0" rpy="0 0 3.1" />
             <geometry>
                 <mesh filename="package://ros_tank_description/meshes/lidarA1.stl" pose="0 0 0" scale="0.00111 0.00111 0.0011"/>
@@ -128,3 +128,86 @@
         </inertial>
     </link>
+     <!-- Joint - camera second servo -->
+    <joint name="camera_servo_second_joint" type="revolute">
+        <origin xyz="0.03 -0.005 0.02" rpy="0 0 0"/>
+        <parent link="camera_servo_first_link"/>
+        <child link="camera_second_servo_link"/>
+        <axis xyz="0 1 0"/>
+        <limit lower="-1.15" upper="1.4" velocity="100" effort="100"/>
+    </joint>
+    <!-- Link - camera second servo -->
+    <link name="camera_second_servo_link">
+        <collision>
+            <origin xyz="0 0 0.01" rpy="0 0 0"/>
+            <geometry>
+                <box size="0.02 0.03 0.03" />
+            </geometry>
+        </collision>
+        <visual>
+            <origin xyz="0 0 0" rpy="0 0 0"/>
+            <geometry>
+                <!-- <box size="0.02 0.03 0.03" /> -->
+                <mesh filename="package://ros_tank_description/meshes/camera_servo_2.stl" pose="0 0 0" scale="0.0011 0.00111 0.0011"/>
+            </geometry>
+        </visual>
+        <inertial>
+            <origin rpy="0 1.5707 1.5707" xyz="0 0 0"/>
+            <mass value="0.05"/>
+            <inertia ixx="1.531666666666667e-05" ixy="0" ixz="0" iyy="1.531666666666667e-05" iyz="0" izz="3.0625000000000006e-05"/>
+        </inertial>
+    </link>
+     <!-- Joint - camera first servo -->
+    <joint name="camera_servo_first_joint" type="revolute">
+        <origin xyz="0.053 0 0" rpy="0 0 0"/>
+        <parent link="link_chassis"/>
+        <child link="camera_servo_first_link"/>
+        <axis xyz="0 0 1"/>
+        <limit lower="-1.15" upper="1.4" velocity="100" effort="100"/>
+    </joint>
+    <!-- Link - camera first servo -->
+    <link name="camera_servo_first_link">
+        <collision>
+            <origin xyz="0 0 -0.005" rpy="0 0 0"/>
+            <geometry>
+                <box size="0.03 0.04 0.03" />
+            </geometry>
+        </collision>
+        <visual>
+            <origin xyz="0 0 0" rpy="0 0 0"/>
+            <geometry>
+                <mesh filename="package://ros_tank_description/meshes/camera_servo_1.stl" pose="0 0 0" scale="0.0011 0.00111 0.0011"/>
+                <!-- <box size="0.03 0.04 0.05" />-->
+            </geometry>
+        </visual>
+        <inertial>
+            <origin rpy="0 1.5707 1.5707" xyz="0 0 0"/>
+            <mass value="0.05"/>
+            <inertia ixx="1.531666666666667e-05" ixy="0" ixz="0" iyy="1.531666666666667e-05" iyz="0" izz="3.0625000000000006e-05"/>
+        </inertial>
+    </link>
+    <!-- Camera -->
+    <joint name="camera_joint" type="fixed">
+        <parent link="camera_second_servo_link"/>
+        <child link="camera_link"/>
+        <origin xyz="0.03 0 0.017" rpy="0 0 0"/>
+    </joint>
+    <link name="camera_link">
+        <collision>
+            <origin xyz="0 0 0" rpy="0 0 0"/>
+            <geometry>
+                <box size="0.02 0.08 0.038"/>
+            </geometry>
+        </collision>
+        <visual>
+            <geometry>
+                <mesh filename="package://ros_tank_description/meshes/camera.stl" pose="0 0 0" scale="0.00111 0.00111 0.0011"/>
+                <!-- <box size="0.02 0.08 0.038"/>-->
+            </geometry>
+        </visual>
+        <inertial>
+            <origin rpy="0 1.5707 1.5707" xyz="0 0 0"/>
+            <mass value="0.05"/>
+            <inertia ixx="1.531666666666667e-05" ixy="0" ixz="0" iyy="1.531666666666667e-05" iyz="0" izz="3.0625000000000006e-05"/>
+        </inertial>
+    </link>
 </robot>

File: ros2_ws/ros_tank_description/urdf/gazebo.xacro (robot description, xacro)
@@ -29,6 +29,6 @@
     </gazebo>
     <gazebo reference="left_wheel">
-        <kp>1000000000000000000000000000.0</kp>
-        <kd>1000000000000000000000000000.0</kd>
+        <kp>10000000.0</kp>
+        <kd>10000000.0</kd>
         <mu1>10.0</mu1>
         <mu2>10.0</mu2>
@@ -36,6 +36,6 @@
     </gazebo>
     <gazebo reference="right_wheel">
-        <kp>1000000000000000000000000000.0</kp>
-        <kd>1000000000000000000000000000.0</kd>
+        <kp>10000000.0</kp>
+        <kd>10000000.0</kd>
         <mu1>10.0</mu1>
         <mu2>10.0</mu2>
@@ -80,5 +80,5 @@
             <scan>
                 <horizontal>
-                    <samples>50</samples>
+                    <samples>150</samples>
                     <resolution>1.0</resolution>
                     <min_angle>-1.0</min_angle>
@@ -86,12 +86,12 @@
                 </horizontal>
                 <vertical>
-                    <samples>50</samples>
+                    <samples>150</samples>
                     <resolution>1.0</resolution>
-                    <min_angle>-1.0</min_angle>
+                    <min_angle>0.0</min_angle>
                     <max_angle>1.0</max_angle>
                 </vertical>
             </scan>
             <range>
-                <min>0.10</min>
+                <min>0.20</min>
                 <max>5.0</max>
                 <resolution>0.01</resolution>
