Commit message: Formatting files

File: ros2_ws/ros_tank_description/urdf/camera_servos_control.xacro (robot description, xacro)
@@ -20,4 +20,26 @@
         </joint>
     </ros2_control>
+<!--   <ros2_control name="camera_controller" type="system">-->
+<!--      <hardware>-->
+<!--        <plugin>ros_tank_hardware/SystemPositionOnlyHardware</plugin>-->
+<!--        <param name="example_param_hw_start_duration_sec">0</param>-->
+<!--        <param name="example_param_hw_stop_duration_sec">3.0</param>-->
+<!--        <param name="example_param_hw_slowdown">10</param>-->
+<!--      </hardware>-->
+<!--      <joint name="camera_servo_first_joint">-->
+<!--        <command_interface name="position">-->
+<!--          <param name="min">-1</param>-->
+<!--          <param name="max">1</param>-->
+<!--        </command_interface>-->
+<!--        <state_interface name="position"/>-->
+<!--      </joint>-->
+<!--      <joint name="camera_servo_second_joint">-->
+<!--        <command_interface name="position">-->
+<!--          <param name="min">-1</param>-->
+<!--          <param name="max">1</param>-->
+<!--        </command_interface>-->
+<!--        <state_interface name="position"/>-->
+<!--      </joint>-->
+<!--    </ros2_control>-->
     <!-- Gazebo's ros2_control plugin -->
     <gazebo>

File: ros_tank_hardware/description/ros2_control/ros_tank.ros2_control.xacro (robot description, xacro)
@@ -7,5 +7,5 @@
         <param name="example_param_hw_start_duration_sec">0</param>
         <param name="example_param_hw_stop_duration_sec">3.0</param>
-        <param name="example_param_hw_slowdown">100</param>
+        <param name="example_param_hw_slowdown">1000</param>
       </hardware>
       <joint name="${prefix}joint1">
